Commit message: implemented forward kinematics

File: robot-urdfs/combined.urdf (robot description, URDF)
Before this commit: robot my_combined_robot, 11 links, 10 joints
Joints:
- removed joint linear_robot
- added joint gantry_robot: type fixed, parent linear_flange, child base_link, origin xyz=0 0 0 rpy=0 0 0

File: robot-urdfs/combined.xacro (robot description, xacro)
@@ -1,10 +1,10 @@
 <?xml version="1.0"?>
 <robot name="my_combined_robot" xmlns:xacro="http://www.ros.org/wiki/xacro">
-  <xacro:include filename="$(find robot_description)/urdf/abb_irb6700_150_320.urdf" />
   <xacro:include filename="$(find robot_description)/urdf/linear_axis.urdf" />
-  <joint name="linear_robot" type="fixed">
+  <joint name="gantry_robot" type="fixed">
     <origin rpy="0 0 0" xyz="0 0 0"/>
     <parent link="linear_flange"/>
     <child link="base_link"/>
   </joint>
+  <xacro:include filename="$(find robot_description)/urdf/abb_irb6700_150_320.urdf" />
 </robot>
